File: PCB/KeysMatrix/KeysMatrix.kicad_pcb (KiCad board)
At the start: 2 copper layers, 123 parts, among them J1 Conn_01x18

Commit message: Complete KeysMatrix
Parts:
- moved D40 59.0 mm to (109.1, 123.6)
- moved D27 55.4 mm to (104.1, 104.7)
- moved D14 54.2 mm to (102.1, 85.5)
- moved J1 52.0 mm to (83.2, 97.5)
- moved D1 50.6 mm to (96.6, 66.6)
- moved D53 50.6 mm to (96.6, 142.6)
- moved D11 44.6 mm to (275.1, 66.6)
- moved D48 44.6 mm to (260.8, 123.6)
- moved D60 44.6 mm to (325.0, 123.6)
- moved S51 44.6 mm to (349.3, 97.6)
- moved S61 44.6 mm to (361.2, 135.7)
- moved D2 44.6 mm to (103.9, 66.6)
- moved D3 44.6 mm to (123.0, 66.6)
- moved D39 44.6 mm to (322.7, 85.6)
- moved D4 44.6 mm to (142.0, 66.6)
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Routing:
- net Column9: track 162.8 -> 836.9 mm, vias 0 -> 2
- net Column8: track 200.0 -> 850.3 mm, vias 0 -> 2
- net Column7: track 0.00 -> 524.2 mm, vias 0 -> 6
- net Column5: track 375.0 -> 892.4 mm
- net Column6: track 449.2 -> 885.3 mm
- net Column10: track 241.2 -> 653.5 mm, vias 0 -> 2
- net Column4: track 300.8 -> 670.3 mm
- net Column11: track 167.1 -> 525.8 mm, vias 0 -> 2
- net Column12: track 96.7 -> 425.9 mm
- net Column13: track 43.1 -> 328.0 mm
- net Column3: track 226.6 -> 452.8 mm
- net Column2: track 152.4 -> 279.3 mm
- net Row4: track 214.0 -> 297.0 mm, vias 0 -> 2
- net Row2: track 237.8 -> 282.2 mm, vias 0 -> 2
- net Row5: track 478.4 -> 521.9 mm
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- added copper zone on B.Cu, net (none)
- added copper zone on F.Cu, net (none)
Other:
- board outline added: 300 x 100 mm
